File: BuckBoostInverter.kicad_pcb (KiCad board)
At the start: 2 copper layers, 100 x 50 mm, 27 parts, among them J1 Conn_01x02_Male, J2 Conn_01x02_Male, Q1 CSD19537Q3, U1 LM5088-1

Commit message: finish layout, generate gerbers
Parts:
- J1, J2: footprint Connector_PinSocket_2.54mm:PinSocket_1x02_P2.54mm_Vertical -> project_lib:PowerPads
- moved C12 63.8 mm to (165.0, 101.4), turned to 180 degrees
- moved C13 54.8 mm to (165.0, 107.4), turned to 180 degrees
- moved C5 53.5 mm to (87.4, 97.1), turned to 90 degrees
- moved C11 45.6 mm to (166.0, 88.2), turned to 270 degrees
- moved J2 41.0 mm to (159.6, 116.4)
- moved C1 40.7 mm to (101.4, 83.9), turned to 90 degrees
- moved R3 28.7 mm to (78.2, 98.9), turned to 90 degrees
- moved C2 22.4 mm to (97.2, 83.8), turned to 90 degrees
- moved R2 19.1 mm to (89.0, 90.1), turned to 270 degrees
- moved C7 18.2 mm to (92.4, 90.0), turned to 270 degrees
- moved R4 17.4 mm to (97.4, 91.9), turned to 270 degrees
- moved D1 17.0 mm to (156.6, 90.3), turned to 0 degrees
- moved R8 16.7 mm to (105.0, 101.4), turned to 270 degrees
- moved R5 16.0 mm to (92.0, 97.0), turned to 90 degrees
- moved C4 14.9 mm to (114.4, 91.1), turned to 270 degrees
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Connections:
- U1 pad 17: Net-(U1-Pad17) -> GND
Routing:
- net GND: track 0.00 -> 192.4 mm, vias 0 -> 17
- net Net-(C11-Pad2): track 0.00 -> 174.3 mm
- net Net-(C1-Pad1): track 0.00 -> 120.5 mm
- net Net-(D1-Pad2): track 0.00 -> 64.9 mm
- net Net-(C8-Pad1): track 0.00 -> 50.8 mm
- net Net-(C5-Pad1): track 0.00 -> 37.6 mm, vias 0 -> 2
- net Net-(Q1-Pad4): track 0.00 -> 31.3 mm, vias 0 -> 2
- net Net-(C6-Pad1): track 0.00 -> 30.0 mm, vias 0 -> 2
- net Net-(R6-Pad2): track 0.00 -> 27.3 mm
- net Net-(C3-Pad1): track 0.00 -> 24.7 mm
- net Net-(C10-Pad1): track 0.00 -> 22.2 mm
- net Net-(C9-Pad2): track 0.00 -> 14.8 mm
- net Net-(C7-Pad1): track 0.00 -> 12.2 mm
- net Net-(C8-Pad2): track 0.00 -> 8.63 mm
- net Net-(R4-Pad1): track 0.00 -> 7.42 mm
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- added copper zone on B.Cu, net GND
- added copper zone on F.Cu, net Net-(C1-Pad1)
- added copper zone on F.Cu, net Net-(C11-Pad2)
Other:
- board text added: "-5.5 Buck Boost Inverter If it works, it was made by Ameet. Otherwise Ben made it"
- board text added: "-5.5V"
- board text added: "GND"
